File: .kicad_pcb.kicad_pcb (KiCad board)
At the start: 2 copper layers, 25 parts, among them K1 CHERRY_ML, K10 CHERRY_ML, K11 CHERRY_ML, K12 CHERRY_ML, K2 CHERRY_ML, K3 CHERRY_ML, K4 CHERRY_ML, K5 CHERRY_ML, K6 CHERRY_ML, K7 CHERRY_ML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

Commit message: working test schematic
Parts:
- D1, D10, D11, D12, D2, D3, D4, D5, D6, D7, D8, D9: footprint FDLL4148 -> 4148_rev2
- moved D12 28.8 mm to (255.3, 179.1)
- moved D3 28.8 mm to (198.1, 179.1)
- moved D9 28.8 mm to (236.2, 179.1)
- moved D5 28.8 mm to (217.2, 179.1)
- moved D11 28.0 mm to (255.3, 161.3)
- moved D2 28.0 mm to (198.1, 161.3)
- moved D8 28.0 mm to (236.2, 161.3)
- moved K12 28.0 mm to (255.3, 170.2)
- moved K3 28.0 mm to (198.1, 170.2)
- moved K9 28.0 mm to (236.2, 170.2)
- moved D4 28.0 mm to (217.2, 161.3)
- moved K5 28.0 mm to (217.2, 170.2)
- moved D1 27.2 mm to (198.1, 143.5)
- moved D10 27.2 mm to (255.3, 143.5)
- moved D7 27.2 mm to (236.2, 143.5)
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Connections:
- D1 pad 2: N-0000030 (its old number) -> N-0000018
- D10 pad 2: N-000003 (its old number) -> N-000002
- D11 pad 2: N-000003 (its old number) -> N-000002
- D12 pad 2: N-000003 (its old number) -> N-000002
- D2 pad 2: N-0000030 (its old number) -> N-0000018
- D3 pad 2: N-0000030 (its old number) -> N-0000018
- P1 pad 4: N-000003 (its old number) -> N-0000018
- P1 pad 5: N-0000013 -> N-000009
- P1 pad 6: N-000009 -> N-0000013
- P1 pad 7: N-0000030 (its old number) -> N-000002
Routing:
- net N-000002: track 0.00 -> 106.0 mm
- net N-000003 (its old number): track 97.8 -> 0.00 mm
- net N-0000013: track 0.00 -> 90.3 mm
- net N-000009: track 0.00 -> 73.0 mm
- net N-0000018: track 0.00 -> 58.7 mm
- net N-0000022: track 86.0 -> 54.0 mm
- net N-000006: track 46.1 -> 15.2 mm
- net N-0000029: track 67.0 -> 36.2 mm
- net N-0000031: track 0.00 -> 14.0 mm
- net N-0000030: track 0.00 -> 14.0 mm
- net N-0000027: track 0.00 -> 14.0 mm
- net N-0000026: track 0.00 -> 14.0 mm
- net N-0000025: track 0.00 -> 14.0 mm
- net N-0000023: track 0.00 -> 14.0 mm
- net N-0000021: track 0.00 -> 14.0 mm
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