File: Atreus_ML.sch (KiCad schematic (older format))
At the start: 25 parts, among them K1 CHERRY_ML, K10 CHERRY_ML, K11 CHERRY_ML, K12 CHERRY_ML, K2 CHERRY_ML, K3 CHERRY_ML, K4 CHERRY_ML, K5 CHERRY_ML, K6 CHERRY_ML, K7 CHERRY_ML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

Commit message: working test schematic
Parts:
- removed D1, D10, D11, D12, D2, D3, D4, D5, D6, D7, D8, D9: DIODE, ~, symbol DIODE
- added D1, D10, D11, D12, D2, D3, D4, D5, D6, D7, D8, D9: 4148, ~, symbol 4148
Connections:
- wire segments 62 -> 61
