File: proto2.kicad_pcb (KiCad board)
At the start: 2 copper layers, 25 parts, among them K1 CHERRY_ML, K10 CHERRY_ML, K11 CHERRY_ML, K12 CHERRY_ML, K2 CHERRY_ML, K3 CHERRY_ML, K4 CHERRY_ML, K5 CHERRY_ML, K6 CHERRY_ML, K7 CHERRY_ML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

Commit message: last update on proto 2 for tonight, saved this time
Parts:
- moved P1 60.7 mm to (172.7, 108.0)
- moved D12 42.4 mm to (227.3, 165.1)
- moved D3 42.2 mm to (170.2, 165.1)
- moved D9 41.3 mm to (208.3, 165.1)
- moved K3 40.9 mm to (170.2, 156.2)
- moved D5 40.9 mm to (189.2, 165.1)
- moved K5 40.0 mm to (189.2, 156.2)
- moved K9 39.5 mm to (208.3, 156.2)
- moved K12 38.2 mm to (227.3, 156.2)
- moved D1 31.2 mm to (170.2, 129.5)
- moved D10 31.2 mm to (227.3, 129.5)
- moved D11 31.2 mm to (227.3, 147.3)
- moved D2 31.2 mm to (170.2, 147.3)
- moved D4 31.2 mm to (189.2, 147.3)
- moved D6 31.2 mm to (189.2, 129.5)
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Routing:
- net N-000002: track 0.00 -> 104.8 mm
- net N-0000013: track 0.00 -> 88.3 mm
- net N-000009: track 0.00 -> 71.7 mm
- net N-0000018: track 0.00 -> 57.5 mm
- net N-0000022: track 0.00 -> 52.7 mm
- net N-0000029: track 0.00 -> 34.9 mm
- net N-000006: track 0.00 -> 14.0 mm
- net N-0000031: track 0.00 -> 14.0 mm
- net N-0000030: track 0.00 -> 14.0 mm
- net N-0000027: track 0.00 -> 14.0 mm
- net N-0000026: track 0.00 -> 14.0 mm
- net N-0000025: track 0.00 -> 14.0 mm
- net N-0000023: track 0.00 -> 14.0 mm
- net N-0000021: track 0.00 -> 14.0 mm
- net N-0000020: track 0.00 -> 14.0 mm
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