File: KiCad/Keyboard/Atreus_ML.kicad_pcb (KiCad board)
At the start: 2 copper layers, 85 parts, among them K1 CHERRY_ML, K10 CHERRY_ML, K11 CHERRY_ML, K12 CHERRY_ML, K13 CHERRY_ML, K14 CHERRY_ML, K15 CHERRY_ML, K16 CHERRY_ML, K17 CHERRY_ML, K18 CHERRY_ML, K19 CHERRY_ML, K2 CHERRY_ML, K20 CHERRY_ML, K21 CHERRY_ML, K22 CHERRY_ML, K23 CHERRY_ML, K24 CHERRY_ML, K25 CHERRY_ML, K26 CHERRY_ML, K27 CHERRY_ML, K28 CHERRY_ML, K29 CHERRY_ML, K3 CHERRY_ML, K30 CHERRY_ML, K31 CHERRY_ML, K32 CHERRY_ML, K33 CHERRY_ML, K34 CHERRY_ML, K35 CHERRY_ML, K36 CHERRY_ML, K37 CHERRY_ML, K38 CHERRY_ML, K39 CHERRY_ML, K4 CHERRY_ML, K40 CHERRY_ML, K41 CHERRY_ML, K42 CHERRY_ML, K5 CHERRY_ML, K6 CHERRY_ML, K7 CHERRY_ML, K8 CHERRY_ML, K9 CHERRY_ML, U1 TEENSY2.0-Compact

Commit message: Edge cuts, they seem ok
Parts:
- moved D4 2.30 mm to (32.0, 127.0)
Routing:
- net Net-(D1-Pad2): track 208.3 -> 207.6 mm
- net Net-(D4-Pad1): track 4.12 -> 3.54 mm
Other:
- board outline added: 252 x 101 mm
Changed lines of the file:
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@@
-(kicad_pcb (version 4) (host pcbnew "(2015-03-15 BZR 5517)-product")
+(kicad_pcb (version 4) (host pcbnew 4.0.2-stable)
   (general
     (links 158)
     (no_connects 0)
-    (area 27.829312 50.549999 273.247628 149.017579)
+    (area 27.829312 50.549999 273.316318 149.349587)
     (thickness 1.6)
-    (drawings 0)
+    (drawings 16)
     (tracks 352)
     (zones 0)
@@
   )
   (module 4148_rev2:4148_rev2 (layer F.Cu)
-    (at 34.244301 127.489549 350)
+    (at 32 127 350)
     (fp_text reference D4 (at 1.27 -2.54 350) (layer F.SilkS) hide
       (effects (font (size 1 1) (thickness 0.15)))
@@
       (net 104 "Net-(K42-Pad1)"))
   )
+  (gr_line (start 37 133) (end 38 134) (angle 90) (layer Edge.Cuts) (width 0.15))
+  (gr_line (start 23 128) (end 37 133) (angle 90) (layer Edge.Cuts) (width 0.15))
+  (gr_line (start 27 108) (end 23 128) (angle 90) (layer Edge.Cuts) (width 0.15))
+  (gr_line (start 26 113) (end 39 49) (angle 90) (layer Edge.Cuts) (width 0.15))
+  (gr_line (start 112 150) (end 113 150) (angle 90) (layer Edge.Cuts) (width 0.15))
+  (gr_line (start 37 133) (end 112 150) (angle 90) (layer Edge.Cuts) (width 0.15))
+  (gr_line (start 136 63) (end 122 49) (angle 90) (layer Edge.Cuts) (width 0.15))
+  (gr_line (start 39 49) (end 122 49) (angle 90) (layer Edge.Cuts) (width 0.15))
+  (gr_line (start 178 49) (end 261 49) (angle 90) (layer Edge.Cuts) (width 0.15))
+  (gr_line (start 164 63) (end 136 63) (angle 90) (layer Edge.Cuts) (width 0.15))
+  (gr_line (start 178 49) (end 164 63) (angle 90) (layer Edge.Cuts) (width 0.15))
+  (gr_line (start 261 49) (end 262 54) (angle 90) (layer Edge.Cuts) (width 0.15))
+  (gr_line (start 275 129) (end 266 132) (angle 90) (layer Edge.Cuts) (width 0.15))
+  (gr_line (start 262 54) (end 275 129) (angle 90) (layer Edge.Cuts) (width 0.15))
+  (gr_line (start 188 150) (end 266 132) (angle 90) (layer Edge.Cuts) (width 0.15))
+  (gr_line (start 112 150) (end 188 150) (angle 90) (layer Edge.Cuts) (width 0.15))
   (segment (start 44.663192 68.401084) (end 45.343892 64.540637) (width 0.5) (layer B.Cu) (net 1))
   (segment (start 44 89) (end 44.266446 89.655086) (width 0.5) (layer B.Cu) (net 2))
@@
   (segment (start 44.266446 89.655086) (end 41 102) (width 0.5) (layer B.Cu) (net 2))
   (segment (start 37 114) (end 36 125) (width 0.5) (layer B.Cu) (net 2))
-  (segment (start 36 125) (end 37.494167 128.062588) (width 0.5) (layer B.Cu) (net 2))
+  (segment (start 36 125) (end 35.249866 127.573039) (width 0.5) (layer B.Cu) (net 2) (status 20))
   (segment (start 40.967131 108.366433) (end 37 114) (width 0.5) (layer B.Cu) (net 2))
   (segment (start 142.38 96.73) (end 142.38 96.62) (width 0.5) (layer B.Cu) (net 2))
@@
   (segment (start 41.870929 84.236792) (end 41.01658 89.082047) (width 0.5) (layer B.Cu) (net 3))
   (segment (start 38.397965 103.932947) (end 37.717265 107.793394) (width 0.5) (layer B.Cu) (net 4))
-  (segment (start 32.925002 123.581538) (end 34.244301 127.489549) (width 0.5) (layer B.Cu) (net 5))
+  (segment (start 32.925002 123.581538) (end 32 127) (width 0.5) (layer B.Cu) (net 5) (status 20))
   (segment (start 64.880291 68.919624) (end 65.560992 65.059177) (width 0.5) (layer B.Cu) (net 6))
   (segment (start 61 103) (end 61.18423 108.884973) (width 0.5) (layer B.Cu) (net 7))

Commit message: Plot of rev 2
Routing:
- net (no net): track 0.00 -> 652.7 mm
Changed lines of the file:
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@@
     (thickness 1.6)
     (drawings 16)
-    (tracks 352)
+    (tracks 364)
     (zones 0)
     (modules 85)
@@
   (gr_line (start 188 150) (end 266 132) (angle 90) (layer Edge.Cuts) (width 0.15))
   (gr_line (start 112 150) (end 188 150) (angle 90) (layer Edge.Cuts) (width 0.15))
+  (segment (start 37 133) (end 112 150) (width 0.5) (layer B.Cu) (net 0))
+  (segment (start 122 49) (end 39 49) (width 0.5) (layer B.Cu) (net 0))
+  (segment (start 164 63) (end 136 63) (width 0.5) (layer B.Cu) (net 0))
+  (segment (start 136 63) (end 122 49) (width 0.5) (layer B.Cu) (net 0))
+  (segment (start 178 49) (end 261 49) (width 0.5) (layer B.Cu) (net 0))
+  (segment (start 266 132) (end 188 150) (width 0.5) (layer B.Cu) (net 0))
+  (segment (start 266 132) (end 275 129) (width 0.5) (layer B.Cu) (net 0))
+  (segment (start 261 49) (end 275 129) (width 0.5) (layer B.Cu) (net 0))
+  (segment (start 178 49) (end 164 63) (width 0.5) (layer B.Cu) (net 0))
+  (segment (start 39 49) (end 23 128) (width 0.5) (layer B.Cu) (net 0))
+  (segment (start 37 133) (end 23 128) (width 0.5) (layer B.Cu) (net 0))
+  (segment (start 112 150) (end 188 150) (width 0.5) (layer B.Cu) (net 0))
   (segment (start 44.663192 68.401084) (end 45.343892 64.540637) (width 0.5) (layer B.Cu) (net 1))
   (segment (start 44 89) (end 44.266446 89.655086) (width 0.5) (layer B.Cu) (net 2))
